File: Hardware/PCBs/GPSBoard/GPSBoard/GPSBoard.kicad_pcb (KiCad board)
At the start: 2 copper layers, 27.4 x 14.8 mm, 8 parts, among them IC1 MAX-M10S-00B, J1 Conn_01x04, J2 Conn_Coaxial

Commit message: Designed GPS board
Parts:
- removed C2: C_Feedthrough, YFF18AC0G475MT0Y0E:YFF18AC
- added D1: ESD9B3.3ST5G, Diode_SMD:D_SOD-923, F.Cu at (81.7, 64.3)
- added D2: LED, LED_SMD:LED_0603_1608Metric_Pad1.05x0.95mm_HandSolder, F.Cu at (97.4, 68.6)
- added D3: LED, LED_SMD:LED_0603_1608Metric_Pad1.05x0.95mm_HandSolder, F.Cu at (97.5, 72.6)
- added D4: LED, LED_SMD:LED_0603_1608Metric_Pad1.05x0.95mm_HandSolder, F.Cu at (101.9, 64.3)
- added FL1: , KiCad:YFF15PC, F.Cu at (74.5, 70.6)
- added H1: MountingHole_Pad, MountingHole:MountingHole_2.2mm_M2_Pad_TopBottom, F.Cu at (73.4, 65.2)
- added H2: MountingHole_Pad, MountingHole:MountingHole_2.2mm_M2_Pad_TopBottom, F.Cu at (105.7, 71.6)
- added R2: 55, Resistor_SMD:R_0603_1608Metric_Pad0.98x0.95mm_HandSolder, F.Cu at (100.9, 68.6)
- added R3: 55, Resistor_SMD:R_0603_1608Metric_Pad0.98x0.95mm_HandSolder, F.Cu at (101.1, 72.6)
- added R4: 55, Resistor_SMD:R_0603_1608Metric_Pad0.98x0.95mm_HandSolder, F.Cu at (104.4, 65.3)
- IC1: value MAX-M10S-00B -> (none); footprint MAX-M10S-00B:MAXM10S00B -> UBLOX_GPS:MAXM10S00B
- J2: footprint Connector_Coaxial:U.FL_Hirose_U.FL-R-SMT-1_Vertical -> Connector_Coaxial:U.FL_Molex_MCRF_73412-0110_Vertical
- L1: value L -> 100s uH
- moved J1 58.9 mm to (110.4, 64.5)
- moved C1 51.1 mm to (99.4, 65.1)
- moved IC1 49.9 mm to (88.9, 68.6)
- moved L1 49.3 mm to (96.9, 65.0), turned to -90 degrees
- moved L2 49.0 mm to (78.6, 69.2)
- moved R1 48.6 mm to (78.6, 71.9), turned to 0 degrees
- moved J2 48.4 mm to (78.5, 65.3), turned to 90 degrees
Connections:
- IC1 pad 13: Net-(IC1-Pad13) -> unconnected-(IC1-Pad13)
- IC1 pad 15: Net-(IC1-Pad15) -> unconnected-(IC1-Pad15)
- IC1 pad 16: Net-(IC1-Pad16) -> unconnected-(IC1-Pad16)
- IC1 pad 17: Net-(IC1-Pad17) -> unconnected-(IC1-Pad17)
- IC1 pad 18: Net-(IC1-Pad18) -> unconnected-(IC1-Pad18)
- IC1 pad 4: Net-(IC1-Pad4) -> unconnected-(IC1-Pad4)
- IC1 pad 5: Net-(IC1-Pad5) -> unconnected-(IC1-Pad5)
- IC1 pad 6: Net-(IC1-Pad6) -> unconnected-(IC1-Pad6)
- IC1 pad 9: Net-(IC1-Pad9) -> unconnected-(IC1-Pad9)
- R1 pad 1: Net-(IC1-Pad14) -> Net-(FL1-Pad3)
- R1 pad 2: Net-(C2-Pad3) -> Net-(IC1-Pad14)
Routing:
- net RX_GPS: track 7.93 -> 19.5 mm
- net TX_GPS: track 7.95 -> 18.9 mm
- net VCC: track 6.25 -> 14.0 mm
- net GND: track 9.33 -> 2.45 mm, vias 107 -> 290
- net Net-(C2-Pad3): track 4.42 -> 0.00 mm
- net Net-(FL1-Pad3): track 0.00 -> 2.86 mm
- net Net-(IC1-Pad14): track 8.62 -> 6.07 mm
- net +3V3: track 5.79 -> 8.32 mm
- net Net-(D1-Pad2): track 7.00 -> 9.34 mm
- net Net-(D3-Pad1): track 0.00 -> 2.01 mm
- net Net-(D4-Pad1): track 0.00 -> 1.70 mm
- net Net-(D2-Pad1): track 0.00 -> 1.66 mm
- net Net-(FL1-Pad1): track 3.27 -> 2.76 mm
Other:
- board size 27.4 x 14.8 mm -> 42.4 x 12.7 mm
- net class Default removed
- board text added: "3V3"
- board text added: "GND"
- board text added: "RX"
- board text added: "TX"
