File: Hardware/PCBs/GPSBoard/GPSBoard/GPSBoard.kicad_sch (KiCad schematic)
At the start: 8 parts, among them IC1 MAX-M10S-00B, J1 Conn_01x04, J2 Conn_Coaxial

Commit message: Designed GPS board
Parts:
- removed C2: C_Feedthrough, YFF18AC0G475MT0Y0E:YFF18AC, symbol Device:C_Feedthrough
- removed IC1: MAX-M10S-00B, MAX-M10S-00B:MAXM10S00B, symbol RF_GPS_new:MAX-M10S-00B
- added D1: ESD9B3.3ST5G, Diode_SMD:D_SOD-923, symbol Diode:ESD9B3.3ST5G
- added D2, D3, D4: LED, LED_SMD:LED_0603_1608Metric_Pad1.05x0.95mm_HandSolder, symbol Device:LED
- added FL1: YFF15PC1A224MT000N, KiCad:YFF15PC, symbol YFF15PC1A224MT000N:YFF15PC1A224MT000N
- added H1, H2: MountingHole_Pad, MountingHole:MountingHole_2.2mm_M2_Pad_TopBottom, symbol Mechanical:MountingHole_Pad
- added IC1: MAX-M10S-00B, UBLOX_GPS:MAXM10S00B, symbol New_Library:MAX-M10S-00B
- added R2, R3, R4: 55, Resistor_SMD:R_0603_1608Metric_Pad0.98x0.95mm_HandSolder, symbol Device:R
- J2: footprint Connector_Coaxial:U.FL_Hirose_U.FL-R-SMT-1_Vertical -> Connector_Coaxial:U.FL_Molex_MCRF_73412-0110_Vertical
- L1: value L -> 100s uH
Connections:
- net +3V3: now also IC1.7 (V_IO), IC1.8 (VCC)
- net GND: now also D1.1 (A1), FL1.2 (GND_1), FL1.4 (GND_2), H1.1, H2.1, IC1.1 (GND_1), IC1.10 (GND_2), IC1.12 (GND_3), R2.2, R3.2, R4.2
- net RX_GPS: now also D2.2 (A), IC1.3 (RXD)
- net TX_GPS: now also D3.2 (A), IC1.2 (TXD)
- net VCC: now also D4.2 (A)
- net at J2.1 (In), L2.1: now also D1.2 (A2), IC1.11 (RF_IN)
- net at L2.2: now also FL1.1 (IN/OUT)
- net at R1.1: now also FL1.3 (OUT/IN)
- net at R1.2: now also IC1.14 (VCC_RF)
- new net: D3.1 (K), R3.1
- new net: D2.1 (K), R2.1
- new net: D4.1 (K), R4.1
Other:
- note added: "MOUNTING"
- note added: "STATUS"
- moved on the sheet: J1, J2, L2, R1
